File: hardware/main_board/main_board.kicad_pcb (KiCad board)
At the start: 4 copper layers, 0 parts

Commit message: Progressed ECAD.
Parts:
- added C1: 100nC, Capacitor_SMD:C_0805_2012Metric, F.Cu at (149.9, 96.3)
- added C10: 10uC, Capacitor_SMD:C_0805_2012Metric, F.Cu at (154.3, 105.3)
- added C11: C, Capacitor_SMD:C_0805_2012Metric, F.Cu at (154.3, 108.3)
- added C12: C, Capacitor_SMD:C_1210_3225Metric, F.Cu at (168.9, 110.9)
- added C2: 10uC, Capacitor_SMD:C_0805_2012Metric, F.Cu at (149.9, 99.3)
- added C3: 100nC, Capacitor_SMD:C_0805_2012Metric, F.Cu at (149.9, 102.3)
- added C4: 100nC, Capacitor_SMD:C_0805_2012Metric, F.Cu at (149.9, 105.3)
- added C5: 10uC, Capacitor_SMD:C_0805_2012Metric, F.Cu at (149.9, 108.3)
- added C6: 10uC, Capacitor_SMD:C_0805_2012Metric, F.Cu at (149.9, 111.3)
- added C7: 10uC, Capacitor_SMD:C_0805_2012Metric, F.Cu at (154.3, 96.3)
- added C8: 100nC, Capacitor_SMD:C_0805_2012Metric, F.Cu at (154.3, 99.3)
- added C9: 100nC, Capacitor_SMD:C_0805_2012Metric, F.Cu at (154.3, 102.3)
- added H1: MountingHole, MountingHole:MountingHole_5.3mm_M5, F.Cu at (121.1, 75.1)
- added H2: MountingHole, MountingHole:MountingHole_5.3mm_M5, F.Cu at (121.1, 87.2)
- added H3: MountingHole, MountingHole:MountingHole_5.3mm_M5, F.Cu at (121.1, 99.4)
- added H4: MountingHole, MountingHole:MountingHole_5.3mm_M5, F.Cu at (121.1, 111.5)
- added J1: Conn_ARM_JTAG_SWD_10, Connector_PinHeader_1.27mm:PinHeader_2x05_P1.27mm_Vertical, F.Cu at (129.2, 107.7)
- added J2: USB_C_Receptacle_USB2.0_16P, Connector_USB:USB_C_Receptacle_HCTL_HC-TYPE-C-16P-01A, F.Cu at (120.8, 125.0)
- added J3: RJ45_Amphenol_RJMG1BD3B8K1ANR, Connector_RJ:RJ45_Amphenol_RJMG1BD3B8K1ANR, F.Cu at (153.3, 74.5)
- added L1: L, Inductor_SMD:L_TaiTech_TMPC1265_13.5x12.5mm, F.Cu at (164.4, 101.8)
- added R3: 27R, Resistor_SMD:R_0201_0603Metric, F.Cu at (116.2, 130.6)
- added R4: 27R, Resistor_SMD:R_0201_0603Metric, F.Cu at (116.2, 132.4)
- added R5: R, Resistor_SMD:R_0805_2012Metric, F.Cu at (163.9, 110.3)
- added R6: R, Resistor_SMD:R_0805_2012Metric, F.Cu at (163.9, 113.2)
- added U1: STM32H563VITx, Package_QFP:LQFP-100_14x14mm_P0.5mm, F.Cu at (136.4, 78.3)
- added U2: TPS54202DDC, Package_TO_SOT_SMD:SOT-23-6, F.Cu at (159.1, 111.2)
- added U3: TLV75533PDBV, Package_TO_SOT_SMD:SOT-23-5, F.Cu at (159.1, 115.8)
- added U4: REF3033, Package_TO_SOT_SMD:SOT-23, F.Cu at (168.6, 115.3)
- added U5: STM32F407VETx, Package_QFP:LQFP-100_14x14mm_P0.5mm, F.Cu at (136.4, 96.8)
- added U6: LAN8742A, Package_DFN_QFN:VQFN-24-1EP_4x4mm_P0.5mm_EP2.5x2.5mm_ThermalVias, F.Cu at (171.4, 72.2)
Other:
- board outline added: 126 x 108.2 mm
