File: hardware/main_board/power_supply.kicad_sch (KiCad schematic)
At the start: 18 parts, among them U12 REF3033, U6 TLV75533PDBV, U7 TPS54202DDC

Commit message: Progressed ECAD.
Parts:
- removed C10, C13: 100nC, Capacitor_SMD:C_0805_2012Metric, symbol Device:C
- removed C11, C12: 10uC, Capacitor_SMD:C_0805_2012Metric, symbol Device:C
- removed C14: C, Capacitor_SMD:C_0805_2012Metric, symbol Device:C
- removed C15: C, Capacitor_SMD:C_1210_3225Metric, symbol Device:C
- removed L1: L, Inductor_SMD:L_TaiTech_TMPC1265_13.5x12.5mm, symbol Device:L
- removed R8, R9: R, Resistor_SMD:R_0805_2012Metric, symbol Device:R
- removed U7: TPS54202DDC, Package_TO_SOT_SMD:SOT-23-6, symbol Regulator_Switching:TPS54202DDC
- renumbered C30 to C1, C32 to C2, C31 to C3, C33 to C4, C35 to C5, C28 to C6, U6 to U3, U12 to U4
Connections:
- net at C1.1, C3.1, U3.1 (IN)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: no longer C2.1, C4.1, U4.1 (IN)
- new net: C2.1, C4.1, U4.1 (IN)
Other:
- note removed: "Vout = 3.645 V (minimum)"
