File: hardware/main_board/mcu.kicad_sch (KiCad schematic)
At the start: 51 parts, among them J6 Conn_ARM_JTAG_SWD_10, J9 USB_C_Receptacle_USB2.0_16P, Q1 BC847, Q2 BC847, Q3 BC847, Q4 BC847, U1 RP2040, U4 W25Q128JVS, U8 W25Q16JVUXIQ, Y1 ABM8-272-T3

Commit message: Progressed ECAD.
Parts:
- removed C1, C2: 15pC, Capacitor_SMD:C_0201_0603Metric, symbol Device:C
- removed C16, C18, C19, C20, C21, C22, C23, C24, C3, C45: 100nC, Capacitor_SMD:C_0201_0603Metric, symbol Device:C
- removed C17, C25, C26, C27: 2u2C, Capacitor_SMD:C_0402_1005Metric, symbol Device:C
- removed C39: 100pC, Capacitor_SMD:C_0402_1005Metric, symbol Device:C
- removed D1, D2, D4, D5: LED, LED_SMD:LED_0805_2012Metric, symbol Device:LED
- removed J9: USB_C_Receptacle_USB2.0_16P, Connector_USB:USB_C_Receptacle_HCTL_HC-TYPE-C-16P-01A, symbol Connector:USB_C_Receptacle_USB2.0_16P
- removed Q1, Q2, Q3, Q4: BC847, Package_TO_SOT_SMD:SOT-23, symbol Transistor_BJT:BC847
- removed R1, R22: 1kR, Resistor_SMD:R_0402_1005Metric, symbol Device:R
- removed R10, R15, R16, R17: 100R, Resistor_SMD:R_0201_0603Metric, symbol Device:R
- removed R11, R12: 27R, Resistor_SMD:R_0201_0603Metric, symbol Device:R
- removed R13, R14: 5k1R, symbol Device:R
- removed R18, R19, R20, R21: 5k1R, Resistor_SMD:R_0402_1005Metric, symbol Device:R
- removed R25, R7: 10kR, symbol Device:R
- removed U1: RP2040, Package_DFN_QFN:QFN-56-1EP_7x7mm_P0.4mm_EP3.2x3.2mm, symbol MCU_RaspberryPi:RP2040
- removed U4: W25Q128JVS, Package_SO:SOIC-8_5.3x5.3mm_P1.27mm, symbol Memory_Flash:W25Q128JVS
- removed U8: W25Q16JVUXIQ, Package_SO:SOIC-8_5.3x5.3mm_P1.27mm, symbol Memory_Flash:W25Q16JVSS
- removed Y1: ABM8-272-T3, Crystal:Crystal_SMD_3225-4Pin_3.2x2.5mm, symbol Device:Crystal_GND24
- added U2: STM32H563VITx, Package_QFP:LQFP-100_14x14mm_P0.5mm, symbol MCU_ST_STM32H5:STM32H563VITx
- renumbered J6 to J1
Connections:
- net RUN: no longer names the net of J1.10 (~{RESET})
- net SWCLK: no longer names the net of J1.4 (SWCLK/TCK)
- net SWD: no longer names the net of J1.2 (SWDIO/TMS)
- new net: U2.10 (VSS), U2.27 (VSS), U2.49 (VSS), U2.74 (VSS), U2.99 (VSS)
- no-connect marks 9 -> 0
Other:
- note removed: "IB = 0.5 mA"
- note removed: "IC = 10 mA"
- note removed: "LIM"
- note removed: "MOTOR"
- note removed: "ON"
- note removed: "Quiescent current analog: 150 µA typical* *temperature sensor disabled (40μA increase if enabled)"
- note removed: "RS485"
- note removed: "SAR ADC Charge bucket filter Low pass filter -3dB Cutoff Frequency: 1,6 MHz"
- note removed: "VBE = 700 mV"
- note removed: "VCEsat = 200 mV"
- moved on the sheet: J1

Commit message: Progressed ECAD.
Parts:
- added J4: Conn_ARM_JTAG_SWD_20, symbol Connector:Conn_ARM_JTAG_SWD_20
Connections:
- net SWDIO: now reaches J1.2 (SWDIO/TMS)
- net SWDIO: now also U2.77 (PA15(JTDI))
- net SWCLK: now reaches J1.4 (SWCLK/TCK)
- net SWCLK: now also U2.76 (PA14(JTCK)
- new net: J4.10 (GND), J4.12 (GND), J4.14 (GND), J4.16 (GND), J4.18 (GND), J4.20 (GND), J4.4 (GND), J4.6 (GND), J4.8 (GND)
